Commit message: Add files via upload

File: ur5_moveit/config/ur5.ros2_control.xacro (robot description, xacro)
@@ -1,54 +1,61 @@
 <?xml version="1.0"?>
 <robot xmlns:xacro="http://www.ros.org/wiki/xacro">
-    <xacro:macro name="ur5_ros2_control" params="name initial_positions_file">
-        <xacro:property name="initial_positions" value="${load_yaml(initial_positions_file)['initial_positions']}"/>
-        <ros2_control name="${name}" type="system">
-            <hardware>
-                <!-- By default, set up controllers for simulation. This won't work on real hardware -->
-                <plugin>mock_components/GenericSystem</plugin>
-            </hardware>
-            <joint name="shoulder_pan_joint">
-                <command_interface name="position"/>
-                <state_interface name="position">
-                  <param name="initial_value">${initial_positions['shoulder_pan_joint']}</param>
-                </state_interface>
-                <state_interface name="velocity"/>
-            </joint>
-            <joint name="shoulder_lift_joint">
-                <command_interface name="position"/>
-                <state_interface name="position">
-                  <param name="initial_value">${initial_positions['shoulder_lift_joint']}</param>
-                </state_interface>
-                <state_interface name="velocity"/>
-            </joint>
-            <joint name="elbow_joint">
-                <command_interface name="position"/>
-                <state_interface name="position">
-                  <param name="initial_value">${initial_positions['elbow_joint']}</param>
-                </state_interface>
-                <state_interface name="velocity"/>
-            </joint>
-            <joint name="wrist_1_joint">
-                <command_interface name="position"/>
-                <state_interface name="position">
-                  <param name="initial_value">${initial_positions['wrist_1_joint']}</param>
-                </state_interface>
-                <state_interface name="velocity"/>
-            </joint>
-            <joint name="wrist_2_joint">
-                <command_interface name="position"/>
-                <state_interface name="position">
-                  <param name="initial_value">${initial_positions['wrist_2_joint']}</param>
-                </state_interface>
-                <state_interface name="velocity"/>
-            </joint>
-            <joint name="wrist_3_joint">
-                <command_interface name="position"/>
-                <state_interface name="position">
-                  <param name="initial_value">${initial_positions['wrist_3_joint']}</param>
-                </state_interface>
-                <state_interface name="velocity"/>
-            </joint>
-        </ros2_control>
-    </xacro:macro>
+  <xacro:macro name="ur5_ros2_control" params="name initial_positions_file">
+    <xacro:property name="initial_positions" value="${xacro.load_yaml(initial_positions_file)['initial_positions']}"/>
+    <ros2_control name="${name}" type="system">
+      <hardware>
+        <!-- By default, set up controllers for simulation. This won't work on real hardware -->
+        <!-- <plugin>mock_components/GenericSystem</plugin> -->
+                      <!-- new added -->
+        <plugin>gazebo_ros2_control/GazeboSystem</plugin>
+      </hardware>
+      <joint name="shoulder_pan_joint">
+          <command_interface name="position"/>
+          <state_interface name="position">
+            <param name="initial_value">${initial_positions['shoulder_pan_joint']}</param>
+          </state_interface>
+          <state_interface name="velocity"/>
+      </joint>
+      <joint name="shoulder_lift_joint">
+          <command_interface name="position"/>
+          <state_interface name="position">
+            <param name="initial_value">${initial_positions['shoulder_lift_joint']}</param>
+          </state_interface>
+          <state_interface name="velocity"/>
+      </joint>
+      <joint name="elbow_joint">
+          <command_interface name="position"/>
+          <state_interface name="position">
+            <param name="initial_value">${initial_positions['elbow_joint']}</param>
+          </state_interface>
+          <state_interface name="velocity"/>
+      </joint>
+      <joint name="wrist_1_joint">
+          <command_interface name="position"/>
+          <state_interface name="position">
+            <param name="initial_value">${initial_positions['wrist_1_joint']}</param>
+          </state_interface>
+          <state_interface name="velocity"/>
+      </joint>
+      <joint name="wrist_2_joint">
+          <command_interface name="position"/>
+          <state_interface name="position">
+            <param name="initial_value">${initial_positions['wrist_2_joint']}</param>
+          </state_interface>
+          <state_interface name="velocity"/>
+      </joint>
+      <joint name="wrist_3_joint">
+          <command_interface name="position"/>
+          <state_interface name="position">
+            <param name="initial_value">${initial_positions['wrist_3_joint']}</param>
+          </state_interface>
+          <state_interface name="velocity"/>
+      </joint>
+    </ros2_control>
+    <gazebo>
+      <plugin name="gazebo_ros2_control" filename="libgazebo_ros2_control.so">
+          <parameters>$(find ur5_moveit)/config/ros_controllers.yaml</parameters>
+      </plugin>
+    </gazebo>
+  </xacro:macro>
 </robot>

File: ur5_moveit/config/ur5.urdf.xacro (robot description, xacro)
@@ -2,12 +2,12 @@
 <robot xmlns:xacro="http://www.ros.org/wiki/xacro" name="ur5">
     <!-- adding gazebo plugin with ros controller -->
-    <gazebo>
+    <!-- <gazebo>
         <plugin name="gazebo_ros2_control" filename="libgazebo_ros2_control.so">
             <parameters>$(find ur5_moveit)/config/ros_controllers.yaml</parameters>
         </plugin>
-    </gazebo>
+    </gazebo> -->
     <!-- Import ur5 urdf file -->
     <xacro:include filename="$(find ur_description)/urdf/ur5_arm.urdf.xacro" />
     <xacro:include filename="ur5.ros2_control.xacro" />
-    <xacro:ur5_ros2_control name="FakeSystem" initial_positions_file="$(find ur5_moveit)/config/initial_positions.yaml"/>
+    <xacro:ur5_ros2_control name="GazeboSystem" initial_positions_file="$(find ur5_moveit)/config/initial_positions.yaml"/>
 </robot>
